Commit message: 新上肢模型 适配

File: src/unilab/assets/robots/dr002/we11/urdf/we11_reviewed.urdf (robot description, URDF)
Before this commit: robot walking_eagle_we11_reviewed, 8 links, 7 joints
Links:
- removed link ancient_link
- added link U1_link, mass 0.00162207; collision box size=0.0121 0.0133 0.0133; visual mesh filename=../meshes_lod/U1_link.STL
- added link U2_link, mass 0.0462933; collision box size=0.394 0.451 0.185; visual mesh filename=../meshes_lod/U2_link.STL
- added link left_wing_link, mass 0.06633; collision box size=0.04 0.36 0.23; visual mesh filename=../meshes_lod/left_wing_link.STL
- added link right_wing_link, mass 0.06633; collision box size=0.04 0.36 0.23; visual mesh filename=../meshes_lod/right_wing_link.STL
- link base_link: mass 1.0693 -> 1.79744014; geometry collision box size=0.11 0.08 0.27; collision box size=0.127969998 0.118299998 0.150000024
Joints:
- removed joint ancient_joint
- added joint U1_joint: type fixed, parent base_link, child U1_link, origin xyz=-0.2383 0.0067051 -0.038129 rpy=-1.5708 -0.48869 0
- added joint U2_joint: type fixed, parent U1_link, child U2_link, origin xyz=0 -0.00673 -0.00665 rpy=1.5708 0 0
- added joint left_wing_joint: type revolute, parent base_link, child left_wing_link, origin xyz=0.14789 0.031025 0.15872 rpy=-1.498663 1.301348 -1.642929, axis 0.46947 0 -0.88295, limit lower=-1.5708 upper=0 effort=5.5 velocity=21.0
- added joint right_wing_joint: type revolute, parent base_link, child right_wing_link, origin xyz=0.14789 -0.031025 0.15872 rpy=1.498663 1.301348 1.642929, axis -0.46947 0 0.88295, limit lower=-1.5708 upper=0 effort=5.5 velocity=21.0

File: src/unilab/assets/robots/dr002/we11/urdf/we11_source.urdf (robot description, URDF)
Before this commit: robot 走地鹰, 8 links, 7 joints
Links:
- removed link ancient_link
- added link U1_link, mass 0.00162207; collision mesh filename=../meshes_lod/U1_link.STL; visual mesh filename=../meshes_lod/U1_link.STL
- added link U2_link, mass 0.0462933; collision mesh filename=../meshes_lod/U2_link.STL; visual mesh filename=../meshes_lod/U2_link.STL
- added link left_wing_link, mass 0.06633; collision mesh filename=../meshes_lod/left_wing_link.STL; visual mesh filename=../meshes_lod/left_wing_link.STL
- added link right_wing_link, mass 0.06506; collision mesh filename=../meshes_lod/right_wing_link.STL; visual mesh filename=../meshes_lod/right_wing_link.STL
- link base_link: mass 1.0693 -> 1.79744014; geometry collision mesh filename=../meshes_lod/base_link.STL; visual mesh filename=../meshes_lod/base_link.STL
- link left_calf_link: geometry collision mesh filename=../meshes_lod/left_calf_link.STL; visual mesh filename=../meshes_lod/left_calf_link.STL
- link left_foot_link: geometry collision mesh filename=../meshes_lod/left_foot_link.STL; visual mesh filename=../meshes_lod/left_foot_link.STL
- link left_thigh_link: mass 0.4724629 -> 0.46123591; geometry collision mesh filename=../meshes_lod/left_thigh_link.STL; visual mesh filename=../meshes_lod/left_thigh_link.STL
- link right_calf_link: geometry collision mesh filename=../meshes_lod/right_calf_link.STL; visual mesh filename=../meshes_lod/right_calf_link.STL
- link right_foot_link: geometry collision mesh filename=../meshes_lod/right_foot_link.STL; visual mesh filename=../meshes_lod/right_foot_link.STL
- link right_thigh_link: mass 0.4724629 -> 0.47246; geometry collision mesh filename=../meshes_lod/right_thigh_link.STL; visual mesh filename=../meshes_lod/right_thigh_link.STL
Joints:
- removed joint ancient_joint
- added joint U1_joint: type revolute, parent base_link, child U1_link, origin xyz=-0.2383 0.0067051 -0.038129 rpy=-1.5708 -0.48869 0, axis 0 0 -1, limit lower=-0.785 upper=0.785 effort=0 velocity=0
- added joint U2_joint: type revolute, parent U1_link, child U2_link, origin xyz=0 -0.00673 -0.00665 rpy=1.5708 0 0, axis 0 0 1, limit lower=-0.785 upper=0.785 effort=0 velocity=0
- added joint left_wing_joint: type revolute, parent base_link, child left_wing_link, origin xyz=0.14789 0.031025 0.15872 rpy=0 1.5708 0, axis 0.46947 0 -0.88295, limit lower=-0.785 upper=0.785 effort=0 velocity=0
- added joint right_wing_joint: type revolute, parent base_link, child right_wing_link, origin xyz=0.14789 -0.030975 0.15872 rpy=0 1.5708 0, axis 0.46947 0 -0.88295, limit lower=-0.785 upper=0.785 effort=0 velocity=0
- joint left_calf_joint: origin xyz=0 0.135800809094126 0.0199999999999967 rpy=0 0 0 -> xyz=0.000196973802905953 0.136029636766888 0.0200000000000024 rpy=0 0 0
- joint left_foot_joint: origin xyz=0 0.149999999999687 0.0572000000000056 rpy=0 0 0 -> xyz=0 0.149999999999687 0.0572 rpy=0 0 0
- joint left_thigh_joint: origin xyz=0.01525 0.0558499999999976 -0.0431991909058736 rpy=-1.5707963267949 0 0 -> xyz=0.0150530261970943 0.0558499999999976 -0.0429703632331118 rpy=-1.5707963267949 0 0

Commit message: feat(archive): update WE11 UniLab bringup

File: src/unilab/assets/robots/dr002/we11/urdf/we11_reviewed.urdf (robot description, URDF)
Before this commit: robot we11_my_version, 11 links, 10 joints
Links:
- link U2_link: geometry collision box size=0.054 0.071 0.030001; visual mesh filename=../meshes_lod/U2_link.STL
- link base_link: geometry collision box size=0.11 0.08 0.11; collision box size=0.12797 0.1183 0.11
- link left_calf_link: geometry collision box size=0.02 0.157276 0.02; visual mesh filename=../meshes_lod/left_calf_link.STL
- link left_thigh_link: geometry collision box size=0.032908 0.1684 0.0228; visual mesh filename=../meshes_lod/left_thigh_link.STL
- link right_calf_link: geometry collision box size=0.02 0.157276 0.02; visual mesh filename=../meshes_lod/right_calf_link.STL
- link right_thigh_link: geometry collision box size=0.032908 0.1684 0.0228; visual mesh filename=../meshes_lod/right_thigh_link.STL
Joints:
- joint left_calf_joint: limit lower=-2.669 upper=-0.17 effort=14.0 velocity=33.0 -> lower=-2.60 upper=-0.17 effort=14.0 velocity=33.0
- joint left_thigh_joint: limit lower=-0.43 upper=1.57 effort=5.5 velocity=21.0 -> lower=-0.13 upper=1.57 effort=5.5 velocity=21.0
- joint right_calf_joint: limit lower=-2.669 upper=-0.17 effort=14.0 velocity=33.0 -> lower=-2.60 upper=-0.17 effort=14.0 velocity=33.0
- joint right_thigh_joint: limit lower=-0.43 upper=1.57 effort=5.5 velocity=21.0 -> lower=-0.13 upper=1.57 effort=5.5 velocity=21.0

Commit message: 策略学不会13.5度以上的倾角，暂时把back课程也屏蔽

File: src/unilab/assets/robots/dr002/we11/urdf/we11_reviewed.urdf (robot description, URDF)
Before this commit: robot we11_my_version, 11 links, 10 joints
Joints:
- joint left_calf_joint: limit lower=-2.60 upper=-0.17 effort=14.0 velocity=33.0 -> lower=-2.522524368 upper=-1.285784060 effort=14.0 velocity=33.0
- joint right_calf_joint: limit lower=-2.60 upper=-0.17 effort=14.0 velocity=33.0 -> lower=-2.522524368 upper=-1.285784060 effort=14.0 velocity=33.0
