Commit message: add:辨识

File: src/unilab/assets/robots/pe03/urdf/pe03.urdf (robot description, URDF)
Before this commit: robot pe03, 9 links, 8 joints
Joints:
- joint L_calf_: limit lower=-1.99 upper=0 effort=14 velocity=27.23 -> lower=-2.02 upper=0.00 effort=14 velocity=27.23
- joint L_hip_: limit lower=0 upper=1.5708 effort=5.5 velocity=10.47 -> lower=-0.20 upper=1.50 effort=5.5 velocity=10.47
- joint L_thigh_: limit lower=-1.658 upper=0 effort=5.5 velocity=10.47 -> lower=-1.44 upper=0.00 effort=5.5 velocity=10.47
- joint R_calf_: limit lower=0 upper=1.99 effort=14 velocity=27.23 -> lower=0.00 upper=2.02 effort=14 velocity=27.23
- joint R_hip_: limit lower=-1.5708 upper=0 effort=5.5 velocity=10.47 -> lower=-1.50 upper=0.20 effort=5.5 velocity=10.47
- joint R_thigh_: limit lower=0 upper=1.658 effort=5.5 velocity=10.47 -> lower=0.00 upper=1.44 effort=5.5 velocity=10.47

File: src/unilab/assets/robots/pe03/urdf/pe03_joint_limits.urdf (robot description, URDF)
Before this commit: robot pe03, 9 links, 8 joints
Joints:
- joint L_calf_: limit lower=-1.99 upper=0 effort=14 velocity=27.23 -> lower=-2.02 upper=0.00 effort=14 velocity=27.23
- joint L_hip_: limit lower=-0.19373154697137057 upper=1.57 effort=5.5 velocity=10.47 -> lower=-0.20 upper=1.50 effort=5.5 velocity=10.47
- joint L_thigh_: limit lower=-1.658 upper=0 effort=5.5 velocity=10.47 -> lower=-1.44 upper=0.00 effort=5.5 velocity=10.47
- joint R_calf_: limit lower=0 upper=1.99 effort=14 velocity=27.23 -> lower=0.00 upper=2.02 effort=14 velocity=27.23
- joint R_hip_: limit lower=-1.57 upper=0.19373154697137057 effort=5.5 velocity=10.47 -> lower=-1.50 upper=0.20 effort=5.5 velocity=10.47
- joint R_thigh_: limit lower=0 upper=1.658 effort=5.5 velocity=10.47 -> lower=0.00 upper=1.44 effort=5.5 velocity=10.47

File: src/unilab/assets/robots/pe04/urdf/pe04.urdf (robot description, URDF)
Before this commit: robot pe04, 9 links, 8 joints
Joints:
- joint L_calf_: limit lower=-1.99 upper=0 effort=14 velocity=27.23 -> lower=-2.02 upper=0.00 effort=14 velocity=27.23
- joint L_hip_: limit lower=-0.19373154697137057 upper=1.57 effort=5.5 velocity=10.47 -> lower=-0.20 upper=1.50 effort=5.5 velocity=10.47
- joint L_thigh_: limit lower=-1.658 upper=0 effort=5.5 velocity=10.47 -> lower=-1.44 upper=0.00 effort=5.5 velocity=10.47
- joint R_calf_: limit lower=0 upper=1.99 effort=14 velocity=27.23 -> lower=0.00 upper=2.02 effort=14 velocity=27.23
- joint R_hip_: limit lower=-1.57 upper=0.19373154697137057 effort=5.5 velocity=10.47 -> lower=-1.50 upper=0.20 effort=5.5 velocity=10.47
- joint R_thigh_: limit lower=0 upper=1.658 effort=5.5 velocity=10.47 -> lower=0.00 upper=1.44 effort=5.5 velocity=10.47

File: src/unilab/assets/robots/pe05/urdf/pe05.urdf (robot description, URDF)
Before this commit: robot pe05, 9 links, 8 joints
Joints:
- joint L_calf_: limit lower=-1.99 upper=0 effort=14 velocity=27.23 -> lower=-2.02 upper=0.00 effort=14 velocity=27.23
- joint L_hip_: limit lower=-0.19373154697137057 upper=1.57 effort=5.5 velocity=10.47 -> lower=-0.20 upper=1.50 effort=5.5 velocity=10.47
- joint L_thigh_: limit lower=-1.658 upper=0 effort=5.5 velocity=10.47 -> lower=-1.44 upper=0.00 effort=5.5 velocity=10.47
- joint R_calf_: limit lower=0 upper=1.99 effort=14 velocity=27.23 -> lower=0.00 upper=2.02 effort=14 velocity=27.23
- joint R_hip_: limit lower=-1.57 upper=0.19373154697137057 effort=5.5 velocity=10.47 -> lower=-1.50 upper=0.20 effort=5.5 velocity=10.47
- joint R_thigh_: limit lower=0 upper=1.658 effort=5.5 velocity=10.47 -> lower=0.00 upper=1.44 effort=5.5 velocity=10.47
